File: Hardware/PIR_USB.kicad_pcb (KiCad board)
At the start: 2 copper layers, 30 x 20 mm, 35 parts, among them J1 USB_C_Receptacle_USB2.0_16P, J2 Conn_01x04, J3 BS412, SW1 SW_Push, U1 STM8S003F3P, U2 CP2102N-Axx-xQFN28, U3 USBLC6-2SC6

Commit message: 310325
Parts:
- moved R3 12.9 mm to (49.8, 48.0), turned to -90 degrees
- moved R4 12.9 mm to (48.2, 48.0), turned to -90 degrees
- moved R9 12.7 mm to (41.5, 41.5)
- moved R5 10.6 mm to (42.8, 43.8), turned to 180 degrees
- moved R13 9.29 mm to (49.2, 37.0)
- moved C1 0.50 mm to (42.8, 45.2)
- moved C2 0.50 mm to (42.8, 46.8)
- moved C3 0.50 mm to (42.8, 48.2)
- moved C4 0.50 mm to (45.8, 45.2)
- moved C8 0.50 mm to (45.8, 46.8)
- moved U3 0.25 mm to (49.0, 44.5)
